Commit message: update params

File: staggerlite_description/urdf/staggerlite_gazebo.xacro (robot description, xacro)
@@ -5,5 +5,5 @@
   <xacro:arg name="lidar_visual"    default="false"/>
   <gazebo reference="base_link">
-    <material>Gazebo/DarkGrey</material>
+    <material>Gazebo/White</material>
   </gazebo>
   <gazebo reference="left_wheel_link">
@@ -73,4 +73,5 @@
   </gazebo> -->
   <gazebo reference="imu_link">
+    <material>Gazebo/Green</material>
     <gravity>true</gravity>
     <sensor name="imu_sensor" type="imu">
@@ -93,5 +94,5 @@
   </gazebo>
   <gazebo reference="lidar_link">
-    <material>Gazebo/FlatBlack</material>
+    <material>Gazebo/Red</material>
     <sensor type="ray" name="lds_lfcd_sensor">
       <pose>0 0 0 0 0 0</pose>
